File: wagon-light/Roco/Eilzugwagen/eilzugwagen.brd (EAGLE design)
At the start: 160 x 100 mm, 47 parts, among them IC2 78L05F, IC3 16F18324-SL, Q1 BC817-25SMD, Q2 BC817-16SMD, Q3 BC817-16SMD, Q4 BC817-16SMD, Q5 BC817-16SMD, Q6 BC817-16SMD, Q7 BC817-16SMD, Q8 BC817-16SMD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

Commit message: misc
Parts:
- removed C6: 10u/35V, rcl:D/7343-31R
- removed LED12, LED13, LED14, LED15, LED16, LED4, LED8: (no value), led:KA-3528ASYC
- removed Q2, Q3: BC817-16SMD, transistor-npn:SOT23-BEC
- removed R12: (no value), rcl:R1206
- moved LED6 170.6 mm to (107.3, 3.62), flipped to the bottom, turned to 90 degrees
- moved LED5 169.7 mm to (112.7, 3.53), flipped to the bottom, turned to 270 degrees
- moved R13 167.5 mm to (101.1, 3.35), turned to 90 degrees
- moved C7 158.5 mm to (110.2, 3.58)
- moved JP3 155.9 mm to (104.0, 3.50)
- moved R15 131.3 mm to (95.7, 3.43), turned to 90 degrees
- moved Q5 129.3 mm to (89.1, 3.50), turned to 180 degrees
- moved R14 129.0 mm to (98.2, 3.39), turned to 90 degrees
- moved LED7 120.5 mm to (90.0, 3.31), flipped to the bottom, turned to 180 degrees
- moved Q1 119.6 mm to (85.5, 3.50), turned to 180 degrees
- moved Q4 119.0 mm to (92.6, 3.50), turned to 180 degrees
- moved D1 117.9 mm to (68.1, 3.50), turned to 180 degrees
- moved R8 116.7 mm to (72.1, 3.42), turned to 90 degrees
- moved R7 114.3 mm to (74.6, 3.42), turned to 90 degrees
- moved C5 113.0 mm to (51.6, 3.39), turned to 90 degrees
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Connections:
- removed net N$10: LED3.C, LED4.A
- removed net N$11: LED7.C, LED8.A
- removed net N$12: LED11.C, LED12.A
- removed net N$13: LED15.C, LED16.A
- removed net N$14: LED16.C, Q2.C
- removed net N$15: LED14.C, LED15.A
- removed net N$17: Q2.E, Q3.B, R12.2
- removed net N$24: LED13.C, LED14.A
- net +15V: no longer C6.+, LED13.A
- net GND: no longer C6.-, Q3.E, R12.1
- net N$30: now also LED3.C; no longer LED4.C
- net N$31: now also LED11.C; no longer LED12.C
- net N$32: now also LED7.C; no longer LED8.C
- net PWM4: no longer Q2.B, Q3.C
Routing:
- net GND: track 0.00 -> 159.2 mm, vias 0 -> 5
- net +15V: track 0.00 -> 132.8 mm, vias 0 -> 5
- net N$26: track 0.00 -> 88.1 mm, vias 0 -> 2
- net N$2: track 0.00 -> 79.9 mm
- net N$25: track 0.00 -> 74.2 mm, vias 0 -> 2
- net +5V: track 0.00 -> 64.1 mm, vias 0 -> 3
- net PWM1: track 0.00 -> 52.3 mm
- net N$31: track 0.00 -> 48.9 mm, vias 0 -> 7
- net N$3: track 0.00 -> 48.6 mm, vias 0 -> 2
- net N$1: track 0.00 -> 48.4 mm, vias 0 -> 1
- net PWM3: track 0.00 -> 41.0 mm
- net PWM2: track 0.00 -> 39.9 mm
- net COMMAND: track 0.00 -> 27.4 mm, vias 0 -> 2
- net 60MA: track 0.00 -> 23.3 mm
- net N$19: track 0.00 -> 19.7 mm
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Other:
- board size 160 x 100 mm -> 116 x 12 mm
