File: wagon-light/Roco/Eilzugwagen/eilzugwagen.sch (EAGLE design)
At the start: 47 parts, among them IC2 78L05F, IC3 16F18324-SL, Q1 BC817-25SMD, Q2 BC817-16SMD, Q3 BC817-16SMD, Q4 BC817-16SMD, Q5 BC817-16SMD, Q6 BC817-16SMD, Q7 BC817-16SMD, Q8 BC817-16SMD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

Commit message: misc
Parts:
- removed C6: 10u/35V, rcl:CPOL-EUD/7343-31R
- removed LED12, LED13, LED14, LED15, LED16, LED4, LED8: (no value), led:LEDKA-3528ASYC
- removed Q2, Q3: BC817-16SMD, transistor-npn:BC817-16SMD
- removed R12: (no value), rcl:R-EU_R1206
Connections:
- removed net N$10: LED3.C, LED4.A
- removed net N$11: LED7.C, LED8.A
- removed net N$12: LED11.C, LED12.A
- removed net N$13: LED15.C, LED16.A
- removed net N$14: LED16.C, Q2.C
- removed net N$15: LED14.C, LED15.A
- removed net N$17: Q2.E, Q3.B, R12.2
- removed net N$24: LED13.C, LED14.A
- net +15V: no longer C6.+, LED13.A
- net GND: no longer C6.-, Q3.E, R12.1
- net N$30: now also LED3.C; no longer LED4.C
- net N$31: now also LED11.C; no longer LED12.C
- net N$32: now also LED7.C; no longer LED8.C
- net PWM4: no longer Q2.B, Q3.C

Commit message: misc
Parts:
- removed Q4, Q5, Q6, Q7, Q8, Q9: BC817-16SMD, transistor-npn:BC817-16SMD
- removed R13, R14, R15: (no value), rcl:R-EU_R1206
- added C4, C6: 10u/35V, rcl:C-EUC3216
- added U1, U2, U3: BCR421U, BCR421U:BCR421U
- C5: device rcl:CPOL-EUA/3216-18R -> rcl:C-EUC3216
- C7, C8: device rcl:CPOL-EUD/7343-31R -> rcl:C-EUC3216
Connections:
- removed net N$18: Q4.E, Q5.B, R13.2
- removed net N$25: Q6.E, Q7.B, R14.2
- removed net N$26: Q8.E, Q9.B, R15.2
- net +15V: now also C4.1, C6.1, C7.1, C8.1; no longer C7.+, C8.+
- net +5V: now also C5.1; no longer C5.+
- net GND: now also C4.2, C5.2, C6.2, C7.2, C8.2, U1.GND, U2.GND, U3.GND; no longer C5.-, C7.-, C8.-, Q5.E, Q7.E, Q9.E, R13.1, R14.1, R15.1
- net N$30: now also U1.OUT@2, U1.OUT@3, U1.OUT@5; no longer Q8.C
- net N$31: now also U3.OUT@2, U3.OUT@3, U3.OUT@5; no longer Q6.C
- net N$32: now also U2.OUT@2, U2.OUT@3, U2.OUT@5; no longer Q4.C
- net PWM1: now also U1.EN; no longer Q8.B, Q9.C
- net PWM2: now also U2.EN; no longer Q4.B, Q5.C
- net PWM3: now also U3.EN; no longer Q6.B, Q7.C
