File: wagon-light/common/50x15/50x15.sch (EAGLE design)
At the start: 55 parts, among them IC2 78L05F, IC3 16F18324-SL, Q1 BC817-25SMD, Q10 BC817-16SMD, Q11 BC817-16SMD, Q12 BC817-16SMD, Q13 BC817-16SMD, Q2 BC817-16SMD, Q3 BC817-16SMD, Q4 BC817-16SMD, Q5 BC817-16SMD, Q6 BC817-16SMD, Q7 BC817-16SMD, Q8 BC817-16SMD, Q9 BC817-16SMD

Commit message: misc
Parts:
- removed C6, C8: 10u/35V, rcl:CPOL-EUD/7343-31R
- removed LED10, LED11, LED12, LED13, LED14, LED15, LED16, LED5, LED6, LED7, LED8, LED9: (no value), led:LEDKA-3528ASYC
- removed LED17, LED18: (no value), led:LED3MM
- removed Q10, Q11, Q12, Q13, Q2, Q3, Q4, Q5, Q6, Q7, Q8, Q9: BC817-16SMD, transistor-npn:BC817-16SMD
- removed R12, R13, R14, R15, R3, R4: (no value), rcl:R-EU_R1206
- added U1: BCR421U, BCR421U:BCR421U
Connections:
- removed net N$11: LED7.C, LED8.A
- removed net N$12: LED11.C, LED12.A
- removed net N$13: LED15.C, LED16.A
- removed net N$14: LED16.C, Q2.C
- removed net N$15: LED14.C, LED15.A
- removed net N$16: LED10.C, LED11.A
- removed net N$17: Q2.E, Q3.B, R12.2
- removed net N$18: Q4.E, Q5.B, R13.2
- removed net N$19: LED6.C, LED7.A
- removed net N$22: LED5.C, LED6.A
- removed net N$23: LED10.A, LED9.C
- removed net N$24: LED13.C, LED14.A
- removed net N$25: Q6.E, Q7.B, R14.2
- removed net N$26: Q8.E, Q9.B, R15.2
- removed net N$27: LED17.C, Q10.C
- removed net N$29: LED18.C, Q12.C
- removed net N$30: LED4.C, Q8.C
- removed net N$31: LED12.C, Q6.C
- removed net N$32: LED8.C, Q4.C
- removed net N$7: Q12.E, Q13.B, R4.2
- removed net PWM1: IC3.RC5, Q8.B, Q9.C
- removed net PWM2: IC3.RC1/AN5, Q4.B, Q5.C
- removed net PWM3: IC3.RC2/AN6, Q6.B, Q7.C
- removed net PWM4: IC3.RC3/AN7, Q2.B, Q3.C
- removed net PWM6: IC3.RC0/AN4, Q12.B, Q13.C
- new net N$8: LED4.C, U1.OUT@2, U1.OUT@3, U1.OUT@5
- net +15V: no longer C6.+, C8.+, LED13.A, LED17.A, LED18.A, LED5.A, LED9.A
- net GND: now also U1.GND; no longer C6.-, C8.-, Q11.E, Q13.E, Q3.E, Q5.E, Q7.E, Q9.E, R12.1, R13.1, R14.1, R15.1, R3.1, R4.1
- net N$6: now also IC3.RC5, U1.EN; no longer Q10.E, Q11.B, R3.2
- net PWM5: no longer Q10.B, Q11.C
Other:
- moved on the sheet: LED1, LED2, LED3, LED4
