File: wagon-light/Roco/Eurofima/eurofima.brd (EAGLE design)
At the start: 155 x 12 mm, 55 parts, among them IC2 78L05F, IC3 16F18324-SL, Q1 BC817-25SMD, Q10 BC817-16SMD, Q11 BC817-16SMD, Q12 BC817-16SMD, Q13 BC817-16SMD, Q2 BC817-16SMD, Q3 BC817-16SMD, Q4 BC817-16SMD, Q5 BC817-16SMD, Q6 BC817-16SMD, Q7 BC817-16SMD, Q8 BC817-16SMD, Q9 BC817-16SMD

Commit message: misc
Parts:
- removed Q10, Q11, Q12, Q13, Q2, Q3, Q4, Q5, Q6, Q7, Q8, Q9: BC817-16SMD, transistor-npn:SOT23-BEC
- removed R12, R13, R14, R15, R3, R4: (no value), rcl:R1206
- added C10, C4, C9: 10u/35V, rcl:C3216
- added U1, U2, U3, U4, U5, U6: BCR421U, BCR421U:SC74-6
- C5: device rcl:A/3216-18R -> rcl:C3216
- C6, C7, C8: device rcl:D/7343-31R -> rcl:C3216
- moved C7 97.6 mm to (137.0, 3.50), turned to 270 degrees
- moved R7 95.2 mm to (127.2, 3.50), turned to 90 degrees
- moved C3 69.8 mm to (122.4, 3.50), turned to 90 degrees
- moved C2 18.6 mm to (30.6, 3.50)
- moved C5 10.0 mm to (52.2, 3.50), turned to 270 degrees
- moved R1 9.06 mm to (46.8, 3.50), turned to 270 degrees
- moved C1 8.43 mm to (57.6, 3.50)
- moved C8 5.72 mm to (117.5, 3.50), turned to 270 degrees
- moved D1 4.92 mm to (110.3, 3.50), turned to 0 degrees
- moved R11 4.80 mm to (41.4, 3.50)
- moved IC2 3.86 mm to (101.9, 3.50)
- moved C6 2.82 mm to (18.8, 3.50), turned to 90 degrees
- moved B1 2.69 mm to (92.6, 3.50)
- moved Q1 1.40 mm to (68.5, 3.50)
- moved IC3 0.10 mm to (77.5, 3.50), turned to 0 degrees
Connections:
- removed net N$17: Q2.E, Q3.B, R12.2
- removed net N$18: Q4.E, Q5.B, R13.2
- removed net N$25: Q6.E, Q7.B, R14.2
- removed net N$26: Q8.E, Q9.B, R15.2
- removed net N$6: Q10.E, Q11.B, R3.2
- removed net N$7: Q12.E, Q13.B, R4.2
- net +15V: now also C10.1, C4.1, C6.1, C7.1, C8.1, C9.1; no longer C6.+, C7.+, C8.+
- net +5V: now also C5.1; no longer C5.+
- net GND: now also C10.2, C4.2, C5.2, C6.2, C7.2, C8.2, C9.2, U1.4, U2.4, U3.4, U4.4, U5.4, U6.4; no longer C5.-, C6.-, C7.-, C8.-, Q11.E, Q13.E, Q3.E, Q5.E, Q7.E, Q9.E, R12.1, R13.1, R14.1, R15.1, R3.1, R4.1
- net N$14: now also U4.2, U4.3, U4.5; no longer Q2.C
- net N$27: now also U5.2, U5.3, U5.5; no longer Q10.C
- net N$29: now also U6.2, U6.3, U6.5; no longer Q12.C
- net N$30: now also U1.2, U1.3, U1.5; no longer Q8.C
- net N$31: now also U3.2, U3.3, U3.5; no longer Q6.C
- net N$32: now also U2.2, U2.3, U2.5; no longer Q4.C
- net PWM1: now also U1.1; no longer Q8.B, Q9.C
- net PWM2: now also U2.1; no longer Q4.B, Q5.C
- net PWM3: now also U3.1; no longer Q6.B, Q7.C
- net PWM4: now also U4.1; no longer Q2.B, Q3.C
- net PWM5: now also U5.1; no longer Q10.B, Q11.C
- net PWM6: now also U6.1; no longer Q12.B, Q13.C
Routing:
- net GND: track 233.3 -> 185.7 mm, vias 7 -> 5
- net +5V: track 66.7 -> 105.8 mm, vias 3 -> 4
- net PWM3: track 36.4 -> 5.82 mm, vias 2 -> 0
- net N$28: track 34.6 -> 63.7 mm, vias 2 -> 0
- net PWM2: track 47.6 -> 20.9 mm, vias 1 -> 2
- net N$25: track 26.1 -> 0.00 mm, vias 1 -> 0
- net N$31: track 28.5 -> 8.67 mm, vias 0 -> 1
- net PWM1: track 58.2 -> 75.5 mm, vias 1 -> 2
- net N$18: track 15.8 -> 0.00 mm, vias 1 -> 0
- net COMMAND: track 62.1 -> 75.6 mm, vias 3 -> 2
- net N$26: track 13.1 -> 0.00 mm, vias 2 -> 0
- net N$5: track 32.9 -> 45.1 mm
- net N$2: track 117.6 -> 129.7 mm, vias 4 -> 2
- net +15V: track 196.9 -> 186.0 mm, vias 4 -> 5
- net N$17: track 10.8 -> 0.00 mm, vias 2 -> 0
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