File: wagon-light/Roco/Eurofima/eurofima.sch (EAGLE design)
At the start: 55 parts, among them IC2 78L05F, IC3 16F18324-SL, Q1 BC817-25SMD, Q10 BC817-16SMD, Q11 BC817-16SMD, Q12 BC817-16SMD, Q13 BC817-16SMD, Q2 BC817-16SMD, Q3 BC817-16SMD, Q4 BC817-16SMD, Q5 BC817-16SMD, Q6 BC817-16SMD, Q7 BC817-16SMD, Q8 BC817-16SMD, Q9 BC817-16SMD

Commit message: misc
Parts:
- removed Q10, Q11, Q12, Q13, Q2, Q3, Q4, Q5, Q6, Q7, Q8, Q9: BC817-16SMD, transistor-npn:BC817-16SMD
- removed R12, R13, R14, R15, R3, R4: (no value), rcl:R-EU_R1206
- added C10, C4, C9: 10u/35V, rcl:C-EUC3216
- added U1, U2, U3, U4, U5, U6: BCR421U, BCR421U:BCR421U
- C5: device rcl:CPOL-EUA/3216-18R -> rcl:C-EUC3216
- C6, C7, C8: device rcl:CPOL-EUD/7343-31R -> rcl:C-EUC3216
Connections:
- removed net N$17: Q2.E, Q3.B, R12.2
- removed net N$18: Q4.E, Q5.B, R13.2
- removed net N$25: Q6.E, Q7.B, R14.2
- removed net N$26: Q8.E, Q9.B, R15.2
- removed net N$6: Q10.E, Q11.B, R3.2
- removed net N$7: Q12.E, Q13.B, R4.2
- net +15V: now also C10.1, C4.1, C6.1, C7.1, C8.1, C9.1; no longer C6.+, C7.+, C8.+
- net +5V: now also C5.1; no longer C5.+
- net GND: now also C10.2, C4.2, C5.2, C6.2, C7.2, C8.2, C9.2, U1.GND, U2.GND, U3.GND, U4.GND, U5.GND, U6.GND; no longer C5.-, C6.-, C7.-, C8.-, Q11.E, Q13.E, Q3.E, Q5.E, Q7.E, Q9.E, R12.1, R13.1, R14.1, R15.1, R3.1, R4.1
- net N$14: now also U4.OUT@2, U4.OUT@3, U4.OUT@5; no longer Q2.C
- net N$27: now also U5.OUT@2, U5.OUT@3, U5.OUT@5; no longer Q10.C
- net N$29: now also U6.OUT@2, U6.OUT@3, U6.OUT@5; no longer Q12.C
- net N$30: now also U1.OUT@2, U1.OUT@3, U1.OUT@5; no longer Q8.C
- net N$31: now also U3.OUT@2, U3.OUT@3, U3.OUT@5; no longer Q6.C
- net N$32: now also U2.OUT@2, U2.OUT@3, U2.OUT@5; no longer Q4.C
- net PWM1: now also U1.EN; no longer Q8.B, Q9.C
- net PWM2: now also U2.EN; no longer Q4.B, Q5.C
- net PWM3: now also U3.EN; no longer Q6.B, Q7.C
- net PWM4: now also U4.EN; no longer Q2.B, Q3.C
- net PWM5: now also U5.EN; no longer Q10.B, Q11.C
- net PWM6: now also U6.EN; no longer Q12.B, Q13.C
