File: wagon-light/Minitrix/Eurofima/eurofima.brd (EAGLE design)
At the start: 152 x 10.5 mm, 40 parts, among them IC2 78L05F, IC3 16F18324-SL, Q1 BC817-25SMD, Q4 BC817-16SMD, Q5 BC817-16SMD, Q6 BC817-16SMD, Q7 BC817-16SMD, Q8 BC817-16SMD, Q9 BC817-16SMD

Commit message: misc
Parts:
- removed Q4, Q5, Q6, Q7, Q8, Q9: BC817-16SMD, transistor-npn:SOT23-BEC
- removed R13, R14, R15: (no value), rcl:R1206
- added U1, U2, U3: BCR421U, BCR421U:SC74-6
- C5: device rcl:A/3216-18R -> rcl:C3216
- C6, C7, C8: device rcl:D/7343-31R -> rcl:C3216
- moved LED12 178.9 mm to (148.6, 5.25), turned to 90 degrees
- moved C8 176.2 mm to (117.8, 5.25), turned to 90 degrees
- moved R11 173.2 mm to (126.1, 5.25), turned to 90 degrees
- moved C2 162.8 mm to (142.1, 5.25), turned to 90 degrees
- moved C7 162.1 mm to (113.8, 5.25), turned to 90 degrees
- moved LED11 160.5 mm to (135.4, 5.25), turned to 270 degrees
- moved C3 156.3 mm to (129.1, 5.25), turned to 90 degrees
- moved LED9 148.5 mm to (109.0, 5.25), turned to 270 degrees
- moved R8 148.3 mm to (105.6, 5.25), turned to 90 degrees
- moved LED10 146.0 mm to (122.2, 5.25), turned to 90 degrees
- moved LED6 133.2 mm to (68.3, 5.25), turned to 270 degrees
- moved R1 132.9 mm to (71.3, 5.25), turned to 270 degrees
- moved LED8 130.5 mm to (95.7, 5.25), turned to 270 degrees
- moved LED5 117.0 mm to (57.1, 5.25), turned to 90 degrees
- moved LED7 114.3 mm to (84.0, 5.25), turned to 90 degrees
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Connections:
- removed net N$18: Q4.E, Q5.B, R13.2
- removed net N$25: Q6.E, Q7.B, R14.2
- removed net N$26: Q8.E, Q9.B, R15.2
- net +15V: now also C6.1, C7.1, C8.1; no longer C6.+, C7.+, C8.+
- net +5V: now also C5.1; no longer C5.+
- net GND: now also C5.2, C6.2, C7.2, C8.2, U1.4, U2.4, U3.4; no longer C5.-, C6.-, C7.-, C8.-, Q5.E, Q7.E, Q9.E, R13.1, R14.1, R15.1
- net N$30: now also U1.2, U1.3, U1.5; no longer Q8.C
- net N$31: now also U3.2, U3.3, U3.5; no longer Q6.C
- net N$32: now also U2.2, U2.3, U2.5; no longer Q4.C
- net PWM1: now also U1.1; no longer Q8.B, Q9.C
- net PWM2: now also U2.1; no longer Q4.B, Q5.C
- net PWM3: now also U3.1; no longer Q6.B, Q7.C
Routing:
- net GND: track 0.00 -> 183.8 mm, vias 0 -> 2
- net +15V: track 0.00 -> 153.4 mm, vias 0 -> 4
- net +5V: track 0.00 -> 143.6 mm, vias 0 -> 4
- net N$2: track 0.00 -> 141.6 mm, vias 0 -> 2
- net PWM3: track 0.00 -> 104.3 mm, vias 0 -> 4
- net N$28: track 0.00 -> 84.3 mm, vias 0 -> 4
- net COMMAND: track 0.00 -> 79.7 mm
- net N$1: track 0.00 -> 62.8 mm, vias 0 -> 1
- net PWM1: track 0.00 -> 56.9 mm
- net PWM2: track 0.00 -> 53.9 mm
- net N$19: track 0.00 -> 16.7 mm
- net N$20: track 0.00 -> 14.6 mm
- net N$16: track 0.00 -> 14.0 mm
- net N$10: track 0.00 -> 14.0 mm
- net N$23: track 0.00 -> 14.0 mm
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