File: loc-decoder/Roco/1044/Decoder-BD62xx/roco1044.brd (EAGLE design)
At the start: 62.2 x 14.5 mm, 31 parts, among them IC1 78L05F, IC2 BD6230F, U1 ATTINY84

Commit message: misc
Connections:
- net N$2 renamed TR-L
- net N$3 renamed TR-R
Changed lines of the file:
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@@
 <?xml version="1.0" encoding="utf-8"?>
 <!DOCTYPE eagle SYSTEM "eagle.dtd">
-<eagle version="9.4.0">
+<eagle version="9.5.2">
 <drawing>
 <settings>
-<setting alwaysvectorfont="yes"/>
+<setting alwaysvectorfont="no"/>
 <setting verticaltext="up"/>
 </settings>
@@
 </elements>
 <signals>
-<signal name="N$2">
+<signal name="TR-L">
 <contactref element="TR-L-1" pad="1"/>
 <contactref element="TR-L-3" pad="1"/>
@@
 <wire x1="31.875" y1="4.5" x2="31.838" y2="4.572" width="0.1524" layer="1"/>
 </signal>
-<signal name="N$3">
+<signal name="TR-R">
 <contactref element="TR-R-1" pad="1"/>
 <contactref element="TR-R-2" pad="1"/>
