File: loc-decoder/Roco/1044/Decoder-BD62xx/roco1044.sch (EAGLE design)
At the start: 31 parts, among them IC1 78L05F, IC2 BD6230F, U1 ATTINY84

Commit message: misc
Connections:
- net N$2 renamed TR-L
- net N$3 renamed TR-R
Changed lines of the file:
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@@
 </busses>
 <nets>
-<net name="N$2" class="0">
+<net name="TR-L" class="0">
 <segment>
 <pinref part="TR-L-1" gate="1" pin="P"/>
@@
 <wire x1="157.48" y1="63.5" x2="157.48" y2="76.2" width="0.1524" layer="91"/>
 <junction x="157.48" y="76.2"/>
+<label x="177.8" y="38.1" size="1.778" layer="95"/>
 </segment>
 </net>
-<net name="N$3" class="0">
+<net name="TR-R" class="0">
 <segment>
 <pinref part="TR-R-1" gate="1" pin="P"/>
@@
 <wire x1="157.48" y1="53.34" x2="157.48" y2="38.1" width="0.1524" layer="91"/>
 <wire x1="157.48" y1="38.1" x2="152.4" y2="38.1" width="0.1524" layer="91"/>
+<label x="157.48" y="48.26" size="1.778" layer="95"/>
 </segment>
 </net>
