File: loc-decoder/Roco/1044/Decoder-BD62xx-Railcom/roco1044.brd (EAGLE design)
At the start: 62.2 x 14.5 mm, 30 parts, among them IC1 78L05F, IC2 BD6230F, U2 ATTINY1614-SSNR, U3 BCR421U

Commit message: misc
Parts:
- removed U3: BCR421U, BCR421U:SC74-6
- C4, C6, C7, C8: device rcl:A/3216-18R -> rcl:CT3528
- moved IC1 32.6 mm to (21.8, 10.5), turned to 180 degrees
- moved U$1 26.9 mm to (25.4, -6.10), turned to 180 degrees
- moved U2 18.7 mm to (14.5, 7.75), turned to 90 degrees
- moved B1 17.3 mm to (31.8, 7.37), turned to 270 degrees
- moved C8 14.7 mm to (53.6, 6.99)
- moved C6 13.6 mm to (44.7, 6.99)
- moved C7 12.7 mm to (49.1, 6.99)
Routing:
- net V+: track 0.00 -> 26.9 mm
- net GND: track 0.00 -> 20.8 mm, vias 0 -> 2
- net TR-L: track 59.7 -> 70.1 mm
- net TR-R: track 60.1 -> 68.5 mm

Commit message: misc
Parts:
- removed J-UPDI: (no value), pinhead:1X03
- added J1: 455-1750-1-ND, SparkFun-Connectors:1X03
- added R7: 22, rcl:R0805
- added R8: 10k, rcl:R0805
- added R9: 6k8, rcl:R0805
- added U$2: BC857BV, Railstars:SOT-666
- added U$3: BC847BV, Railstars:SOT-666
- R1, R11, R2, R3, R4, R5, R6: device rcl:R0603 -> rcl:R0805
- moved C4 40.0 mm to (52.8, 11.4), turned to 0 degrees
- moved IC1 22.9 mm to (44.7, 10.2), turned to 270 degrees
- moved C3 21.8 mm to (22.5, 11.3), turned to 90 degrees
- moved R6 21.7 mm to (54.9, 7.24), turned to 90 degrees
- moved R11 21.3 mm to (17.7, 11.3), turned to 270 degrees
- moved R5 19.4 mm to (56.9, 7.24), turned to 270 degrees
- moved U$1 17.8 mm to (25.8, 11.7), turned to 0 degrees
- moved R1 17.5 mm to (57.9, 4.10)
- moved C1 17.0 mm to (20.1, 11.3), turned to 90 degrees
- moved R3 13.1 mm to (4.65, 10.4)
- moved R2 10.6 mm to (57.9, 10.4)
- moved R4 9.92 mm to (4.61, 4.09)
- moved C8 3.10 mm to (51.8, 4.45)
- moved C7 2.90 mm to (47.8, 4.45)
- moved C6 2.74 mm to (43.7, 4.45)
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Connections:
- new net N$1: R9.2, U$3.P$5
- new net N$14: R8.1, U$2.P$5, U$2.P$6
- new net N$3: R9.1, U$2.P$3, U$3.P$1, U$3.P$2
- new net RAILCOM: R8.2, U2.11
- net +5V: now also J1.2, R7.2, U$2.P$1; no longer J-UPDI.2
- net GND: now also J1.1, U$3.P$4; no longer J-UPDI.1
- net N$12: now also R7.1, U$2.P$2, U$2.P$4; no longer U2.11
- net RST: now also J1.3; no longer J-UPDI.3
- net TR-L: now also U$3.P$6
- net TR-R: now also U$3.P$3
Routing:
- net V+: track 26.9 -> 24.9 mm
- net TR-R: track 68.5 -> 66.5 mm
- net N$7: track 0.00 -> 1.96 mm
- net N$6: track 0.00 -> 1.88 mm
- net TR-L: track 70.1 -> 71.9 mm
- net GND: track 20.8 -> 19.2 mm

Commit message: misc
Connections:
- removed net N$16: U2.9
- removed net N$18: U2.7
- removed net N$19: U2.6
- removed net N$2: U2.2
- removed net RST: J1.3
- net RST/UDPI: now also J1.3
Routing:
- net N$5: track 0.00 -> 92.7 mm, vias 0 -> 3
- net +5V: track 0.00 -> 77.8 mm, vias 0 -> 9
- net N$8: track 0.00 -> 77.0 mm, vias 0 -> 3
- net BEMF: track 0.00 -> 56.8 mm, vias 0 -> 3
- net GND: track 19.2 -> 71.9 mm, vias 2 -> 6
- net REVERSE: track 0.00 -> 51.6 mm, vias 0 -> 4
- net V+: track 24.9 -> 76.3 mm, vias 0 -> 1
- net FORWARD: track 0.00 -> 30.7 mm, vias 0 -> 4
- net TR-L: track 71.9 -> 100.8 mm, vias 2 -> 6
- net LIGHT-B: track 0.00 -> 24.8 mm, vias 0 -> 2
- net N$3: track 0.00 -> 24.0 mm, vias 0 -> 2
- net N$11: track 5.33 -> 28.8 mm, vias 0 -> 2
- net LIGHT-F: track 0.00 -> 19.6 mm, vias 0 -> 2
- net N$4: track 2.99 -> 21.8 mm, vias 0 -> 2
- net RST/UDPI: track 0.00 -> 14.5 mm, vias 0 -> 1
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