File: loc-decoder/Roco/1044/Decoder-BD62xx-Railcom/roco1044.brd (EAGLE design)
At the start: 62.2 x 14.5 mm, 34 parts, among them IC1 78L05F, IC2 BD6230F, J1 455-1750-1-ND, U2 ATTINY1614-SSNR

Commit message: misc
Connections:
- net N$11 renamed M-L
- net N$4 renamed M-R
Changed lines of the file:
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@@
 <wire x1="1.8288" y1="4.7244" x2="1.736" y2="4.77" width="0.1524" layer="1"/>
 </signal>
-<signal name="N$4">
+<signal name="M-R">
 <contactref element="M-R" pad="1"/>
 <contactref element="R6" pad="2"/>
@@
 <via x="41.3004" y="11.1252" extent="1-16" drill="0.3"/>
 </signal>
-<signal name="N$11">
+<signal name="M-L">
 <contactref element="M-L" pad="1"/>
 <contactref element="IC2" pad="1"/>
