File: loc-decoder/Roco/1044/Decoder-BD62xx-Railcom/roco1044.sch (EAGLE design)
At the start: 30 parts, among them IC1 78L05F, IC2 BD6230F, U2 ATTINY1614-SSNR, U3 BCR421U

Commit message: misc
Parts:
- removed U3: BCR421U, BCR421U:BCR421U
- C4, C6, C7, C8: device rcl:CPOL-EUA/3216-18R -> rcl:CPOL-EUCT3528
Changed lines of the file:
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@@
 <part name="GND9" library="supply1" library_urn="urn:adsk.eagle:library:371" deviceset="GND" device=""/>
 <part name="P+8" library="supply1" library_urn="urn:adsk.eagle:library:371" deviceset="V+" device=""/>
-<part name="C6" library="rcl" library_urn="urn:adsk.eagle:library:334" deviceset="CPOL-EU" device="A/3216-18R" package3d_urn="urn:adsk.eagle:package:23410/2" value="&gt;1u, &gt;30V"/>
-<part name="C7" library="rcl" library_urn="urn:adsk.eagle:library:334" deviceset="CPOL-EU" device="A/3216-18R" package3d_urn="urn:adsk.eagle:package:23410/2" value="&gt;1u, &gt;30V"/>
-<part name="C8" library="rcl" library_urn="urn:adsk.eagle:library:334" deviceset="CPOL-EU" device="A/3216-18R" package3d_urn="urn:adsk.eagle:package:23410/2" value="&gt;1u, &gt;30V"/>
-<part name="C4" library="rcl" library_urn="urn:adsk.eagle:library:334" deviceset="CPOL-EU" device="A/3216-18R" package3d_urn="urn:adsk.eagle:package:23410/2" value="&gt;10u, &gt;6V"/>
+<part name="C6" library="rcl" library_urn="urn:adsk.eagle:library:334" deviceset="CPOL-EU" device="CT3528" package3d_urn="urn:adsk.eagle:package:23325/2" value="&gt;1u, &gt;30V"/>
+<part name="C7" library="rcl" library_urn="urn:adsk.eagle:library:334" deviceset="CPOL-EU" device="CT3528" package3d_urn="urn:adsk.eagle:package:23325/2" value="&gt;1u, &gt;30V"/>
+<part name="C8" library="rcl" library_urn="urn:adsk.eagle:library:334" deviceset="CPOL-EU" device="CT3528" package3d_urn="urn:adsk.eagle:package:23325/2" value="&gt;1u, &gt;30V"/>
+<part name="C4" library="rcl" library_urn="urn:adsk.eagle:library:334" deviceset="CPOL-EU" device="CT3528" package3d_urn="urn:adsk.eagle:package:23325/2" value="&gt;10u, &gt;6V"/>
 <part name="U2" library="ATTINY1614-SSNR" deviceset="ATTINY1614-SSNR" device=""/>
-<part name="U3" library="BCR421U" deviceset="BCR421U" device=""/>
 <part name="J-UPDI" library="pinhead" library_urn="urn:adsk.eagle:library:325" deviceset="PINHD-1X3" device="" package3d_urn="urn:adsk.eagle:package:22458/2"/>
 </parts>
@@
 <attribute name="VALUE" x="88.9" y="51.88" size="2.0828" layer="96" ratio="10" rot="SR0"/>
 </instance>
-<instance part="U3" gate="G$1" x="17.78" y="111.76" smashed="yes">
-<attribute name="NAME" x="7.6038" y="120.664159375" size="1.78083125" layer="95"/>
-<attribute name="VALUE" x="7.6185" y="100.9634" size="1.778259375" layer="96"/>
-</instance>
 <instance part="J-UPDI" gate="A" x="200.66" y="96.52" smashed="yes">

Commit message: misc
Parts:
- removed J-UPDI: (no value), pinhead:PINHD-1X3
- added J1: 455-1750-1-ND, SparkFun-Connectors:CONN_03
- added R7: 22, rcl:R-EU_R0805
- added R8: 10k, rcl:R-EU_R0805
- added R9: 6k8, rcl:R-EU_R0805
- added U$2: BC857BV, Railstars:BC857BV
- added U$3: BC847BV, Railstars:BC847BV
- R1, R11, R2, R3, R4, R5, R6: device rcl:R-EU_R0603 -> rcl:R-EU_R0805
Connections:
- new net N$1: R9.2, U$3G$2.B
- new net N$14: R8.1, U$2G$1.C, U$2G$2.B
- new net N$3: R9.1, U$2G$2.C, U$3G$1.B, U$3G$1.E
- new net RAILCOM: R8.2, U2.PA1
- net +5V: now also J1.2, R7.2, U$2G$1.E; no longer J-UPDI.2
- net GND: now also J1.1, U$3G$2.E; no longer J-UPDI.1
- net N$12: now also R7.1, U$2G$1.B, U$2G$2.E; no longer U2.PA1
- net RST: now also J1.3; no longer J-UPDI.3
- net TR-L: now also U$3G$1.C
- net TR-R: now also U$3G$2.C

Commit message: misc
Connections:
- removed net N$16: U2.PB0
- removed net N$18: U2.PB2/OSC2
- removed net N$19: U2.PB3/OSC1
- removed net N$2: U2.PA4
- removed net RST: J1.3
- net RST/UDPI: now also J1.3
Changed lines of the file:
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@@
-</segment>
-</net>
-<net name="RST" class="0">
-<segment>
-<wire x1="167.64" y1="93.98" x2="198.12" y2="93.98" width="0.1524" layer="91"/>
-<label x="175.26" y="93.98" size="1.778" layer="95"/>
-<pinref part="J1" gate="J$1" pin="3"/>
 </segment>
 </net>
@@
 <wire x1="185.42" y1="73.66" x2="170.18" y2="73.66" width="0.1524" layer="91"/>
 <label x="170.18" y="73.66" size="1.778" layer="95"/>
-</segment>
-</net>
-<net name="N$2" class="0">
-<segment>
-<pinref part="U2" gate="G$1" pin="PA4"/>
-<wire x1="83.82" y1="68.58" x2="71.12" y2="68.58" width="0.1524" layer="91"/>
 </segment>
 </net>
@@
 </segment>
 </net>
-<net name="N$16" class="0">
-<segment>
-<pinref part="U2" gate="G$1" pin="PB0"/>
-<wire x1="129.54" y1="73.66" x2="144.78" y2="73.66" width="0.1524" layer="91"/>
-</segment>
-</net>
-<net name="N$18" class="0">
-<segment>
-<pinref part="U2" gate="G$1" pin="PB2/OSC2"/>
-<wire x1="129.54" y1="68.58" x2="144.78" y2="68.58" width="0.1524" layer="91"/>
-</segment>
-</net>
-<net name="N$19" class="0">
-<segment>
-<pinref part="U2" gate="G$1" pin="PB3/OSC1"/>
-<wire x1="129.54" y1="66.04" x2="144.78" y2="66.04" width="0.1524" layer="91"/>
-</segment>
-</net>
 <net name="RST/UDPI" class="0">
 <segment>
@@
 <label x="71.12" y="78.74" size="1.778" layer="95"/>
 </segment>
+<segment>
+<pinref part="J1" gate="J$1" pin="3"/>
+<wire x1="198.12" y1="93.98" x2="182.88" y2="93.98" width="0.1524" layer="91"/>
+<label x="182.88" y="93.98" size="1.778" layer="95"/>
+</segment>
 </net>

Commit message: misc
Connections:
- net N$11 renamed M-L
- net N$4 renamed M-R
Changed lines of the file:
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@@
 </segment>
 </net>
-<net name="N$4" class="0">
+<net name="M-R" class="0">
 <segment>
 <pinref part="M-R" gate="1" pin="P"/>
@@
 <wire x1="162.56" y1="-7.62" x2="152.4" y2="-7.62" width="0.1524" layer="91"/>
 <junction x="162.56" y="-7.62"/>
+<label x="157.48" y="-7.62" size="1.778" layer="95"/>
 </segment>
 </net>
-<net name="N$11" class="0">
+<net name="M-L" class="0">
 <segment>
 <pinref part="M-L" gate="1" pin="P"/>
@@
 <wire x1="162.56" y1="5.08" x2="162.56" y2="2.54" width="0.1524" layer="91"/>
 <junction x="162.56" y="2.54"/>
+<label x="157.48" y="-5.08" size="1.778" layer="95"/>
 </segment>
 </net>
