File: loc-decoder/Spectrum/GE Dash 8-40CW-Railcom/dash8_40cw.brd (EAGLE design)
At the start: 95 x 10.4 mm, 27 parts, among them IC1 78L05F, IC2 BD6230F, U1 ATTINY84

Commit message: misc
Parts:
- removed C2: 100n, rcl:C0805
- removed D1: MM3Z27VT1G, diode:SOD323-R
- removed J1: (no value), SparkFun-Connectors:1X06_1.27MM
- removed U1: ATTINY84, SparkFun-IC-Microcontroller:SO14
- added J2: 455-1750-1-ND, SparkFun-Connectors:1X03
- added R13: 22, rcl:R0805
- added R14: 10k, rcl:R0805
- added R15: 6k8, rcl:R0805
- added U$3: BC857BV, Railstars:SOT-666
- added U$4: BC847BV, Railstars:SOT-666
- added U2: ATTINY1614-SSNR, ATTINY1614-SSNR:SOIC127P600X175-14N
- moved C3 56.9 mm to (61.6, 5.29), turned to 270 degrees
- moved B1 47.4 mm to (24.8, 5.19), turned to 270 degrees
- moved R5 25.6 mm to (44.0, 7.98), turned to 0 degrees
- moved U$1 18.0 mm to (45.0, 2.58)
- moved C1 14.9 mm to (40.6, 2.07), turned to 180 degrees
- moved R6 9.61 mm to (40.1, 7.98), turned to 0 degrees
- moved R11 4.76 mm to (14.5, 8.52), turned to 180 degrees
- moved IC1 1.17 mm to (49.5, 6.32), turned to 180 degrees
- moved IC2 0.61 mm to (35.8, 5.20)
- moved R4 0.51 mm to (93.1, 8.73)
- moved C7 0.41 mm to (89.1, 5.30)
- moved C4 0.22 mm to (76.6, 5.30)
- moved C5 0.22 mm to (84.9, 5.30)
- moved C6 0.14 mm to (80.7, 5.30)
- moved R2 0.10 mm to (2.27, 8.73)
Connections:
- net N$11 renamed M-L
- net N$4 renamed M-R
- removed net MISO: J1.5, U$1.P$5, U1.8
- removed net MOSI: J1.4, U$1.P$2, U1.7
- removed net N$12: R11.1, U1.11
- removed net N$2: B1.~1, R11.2, TR-L-1.1, TR-L-2.1
- removed net N$3: B1.~2, TR-R-1.1, TR-R-2.1
- removed net RST: J1.3, U1.4
- removed net SCK: J1.6, U1.9
- new net COMMAND: R11.1, U2.12
- new net LIGHT-B: U$1.P$5, U2.4
- new net LIGHT-F: U$1.P$2, U2.3
- new net N$18: R15.2, U$4.P$5
- new net N$19: R15.1, U$3.P$3, U$4.P$1, U$4.P$2
- new net N$20: R13.1, U$3.P$2, U$3.P$4
- new net N$21: R14.1, U$3.P$5, U$3.P$6
- new net RAILCOM: R14.2, U2.11
- new net RST/UDPI: J2.3, U2.10
- new net TR-L: B1.~1, R11.2, TR-L-1.1, TR-L-2.1, U$4.P$6
- new net TR-R: B1.~2, TR-R-1.1, TR-R-2.1, U$4.P$3
- net +5V: now also J2.2, R13.2, U$3.P$1, U2.1; no longer C2.2, J1.2, U1.1
- net BEMF: now also U2.13; no longer U1.10
- net FORWARD: now also U2.5; no longer U1.6
- net GND: now also J2.1, U$4.P$4, U2.14; no longer C2.1, D1.A, J1.1, U1.14
- net REVERSE: now also U2.8; no longer U1.3
- net V+: no longer D1.C
Routing:
- net N$3: track 60.9 -> 0.00 mm, vias 3 -> 0
- net RST/UDPI: track 0.00 -> 59.7 mm, vias 0 -> 2
- net N$21: track 0.00 -> 58.8 mm, vias 0 -> 2
- net COMMAND: track 0.00 -> 58.0 mm, vias 0 -> 2
- net N$2: track 57.6 -> 0.00 mm, vias 2 -> 0
- net TR-L: track 0.00 -> 53.6 mm
- net TR-R: track 0.00 -> 53.2 mm
- net N$20: track 0.00 -> 49.1 mm, vias 0 -> 2
- net MISO: track 42.4 -> 0.00 mm, vias 1 -> 0
- net GND: track 152.1 -> 182.1 mm, vias 9 -> 4
- net +5V: track 135.7 -> 107.7 mm, vias 6 -> 3
- net LIGHT-B: track 0.00 -> 25.6 mm, vias 0 -> 2
- net LIGHT-F: track 0.00 -> 25.5 mm, vias 0 -> 2
- net MOSI: track 22.7 -> 0.00 mm, vias 2 -> 0
- net N$5: track 71.5 -> 51.9 mm
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Other:
- board text added: "https://github.com/stb49078/nscale-adapter-decoder"
