File: loc-decoder/Spectrum/GE Dash 8-40CW-Railcom/dash8_40cw.sch (EAGLE design)
At the start: 27 parts, among them IC1 78L05F, IC2 BD6230F, U1 ATTINY84

Commit message: misc
Parts:
- removed C2: 100n, rcl:C-EUC0805
- removed D1: MM3Z27VT1G, diode:DIODE-SOD323-R
- removed J1: (no value), SparkFun-Connectors:CONN_061.27MM
- removed U1: ATTINY84, SparkFun-IC-Microcontroller:ATTINY84
- added J2: 455-1750-1-ND, SparkFun-Connectors:CONN_03
- added R13: 22, rcl:R-EU_R0805
- added R14: 10k, rcl:R-EU_R0805
- added R15: 6k8, rcl:R-EU_R0805
- added U$3: BC857BV, Railstars:BC857BV
- added U$4: BC847BV, Railstars:BC847BV
- added U2: ATTINY1614-SSNR, ATTINY1614-SSNR:ATTINY1614-SSNR
Connections:
- net N$11 renamed M-L
- net N$4 renamed M-R
- removed net MISO: J1.5, U$1G$2.G, U1.(PCINT5/OC1B/MISO/DO/ADC5)PA5
- removed net MOSI: J1.4, U$1G$1.G, U1.(PCINT6/OC1A/SDA/MOSI/ADC6)PA6
- removed net N$12: R11.1, U1.(PCINT2/AIN1/ADC2)PA2
- removed net N$2: B1.AC1, R11.2, TR-L-1.P, TR-L-2.P
- removed net N$3: B1.AC2, TR-R-1.P, TR-R-2.P
- removed net RST: J1.3, U1.(PCINT11/~RESET/DW)PB3
- removed net SCK: J1.6, U1.(PCINT4/T1/SCL/USCK/ADC4)PA4
- new net COMMAND: R11.1, U2.PA2
- new net LIGHT-B: U$1G$2.G, U2.PA6
- new net LIGHT-F: U$1G$1.G, U2.PA5
- new net N$18: R15.2, U$4G$2.B
- new net N$19: R15.1, U$3G$2.C, U$4G$1.B, U$4G$1.E
- new net N$20: R13.1, U$3G$1.B, U$3G$2.E
- new net N$21: R14.1, U$3G$1.C, U$3G$2.B
- new net RAILCOM: R14.2, U2.PA1
- new net RST/UDPI: J2.3, U2.PA0/!RESET!/UDPI
- new net TR-L: B1.AC1, R11.2, TR-L-1.P, TR-L-2.P, U$4G$1.C
- new net TR-R: B1.AC2, TR-R-1.P, TR-R-2.P, U$4G$2.C
- net +5V: now also J2.2, R13.2, U$3G$1.E, U2.VDD; no longer C2.2, J1.2, U1.VCC
- net BEMF: now also U2.PA3/EXTCLK; no longer U1.(PCINT3/T0/ADC3)PA3
- net FORWARD: now also U2.PA7; no longer U1.(PCINT7/ICP/OC0B/ADC7)PA7
- net GND: now also J2.1, U$4G$2.E, U2.GND; no longer C2.1, D1.A, J1.1, U1.GND
- net REVERSE: now also U2.PB1; no longer U1.(PCINT9/XTAL2)PB1
- net V+: no longer D1.C
Other:
- note removed: "ZXMHC3F381N8TC or DMHC3025LSD"
