File: loc-decoder/Roco/1044/NEM-651 Adapter/roco1044.brd (EAGLE design)
At the start: 62.2 x 14.5 mm, 16 parts

Commit message: misc
Connections:
- net N$11 renamed M-L
- net N$4 renamed M-R
Other:
- board text added: "Motor Right / Orange"
- board text added: "https://github.com/stb49078/nscale-adapter-decoder"
Changed lines of the file:
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@@
 <?xml version="1.0" encoding="utf-8"?>
 <!DOCTYPE eagle SYSTEM "eagle.dtd">
-<eagle version="9.3.0">
+<eagle version="9.5.2">
 <drawing>
 <settings>
@@
 <wire x1="43.5" y1="2.95" x2="32" y2="2.95" width="0.1524" layer="46"/>
 <wire x1="32" y1="2.95" x2="32" y2="11.5" width="0.1524" layer="46"/>
+<text x="28" y="11" size="0.4064" layer="25" rot="R180">Motor Right / Orange</text>
+<text x="41" y="12" size="0.6096" layer="26" rot="MR0">https://github.com/stb49078/nscale-adapter-decoder</text>
 </plain>
 <attributes>
@@
 <wire x1="6.45" y1="4.71" x2="6.484" y2="4.744" width="0.254" layer="1"/>
 </signal>
-<signal name="N$4">
+<signal name="M-R">
 <contactref element="651" pad="1"/>
 <contactref element="M-R" pad="1"/>
@@
 <wire x1="29.95" y1="13" x2="29.95" y2="10.355" width="0.6096" layer="1"/>
 </signal>
-<signal name="N$11">
+<signal name="M-L">
 <contactref element="651" pad="2"/>
 <contactref element="M-L" pad="1"/>
@@
 <mfgpreviewcolor name="substratecolor" color="0xFF786E46"/>
 </mfgpreviewcolors>
+<errors>
+</errors>
 </board>
 </drawing>
