File: loc-decoder/Roco/BR215/br215.brd (EAGLE design)
At the start: 74 x 9.2 mm, 13 parts

Commit message: misc
Parts:
- added BLAU: (no value), pinhead:1X01
Connections:
- net N$1: now also BLAU.1
Routing:
- net N$2: track 78.0 -> 76.3 mm
- net N$3: track 82.1 -> 80.3 mm
Other:
- board text added: "Motor-R"
- board text added: "https://github.com/stb49078/nscale-adapter-decoder"
Changed lines of the file:
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@@
 <?xml version="1.0" encoding="utf-8"?>
 <!DOCTYPE eagle SYSTEM "eagle.dtd">
-<eagle version="9.4.0">
+<eagle version="9.5.2">
 <drawing>
 <settings>
@@
 <wire x1="65.5" y1="7" x2="65.5" y2="8" width="0.1524" layer="20"/>
 <wire x1="65.5" y1="8" x2="74" y2="8" width="0.1524" layer="20"/>
+<text x="16.7" y="6.6" size="0.8128" layer="25">Motor-R</text>
+<text x="30.4" y="0.3" size="0.6096" layer="25">https://github.com/stb49078/nscale-adapter-decoder</text>
 </plain>
 <attributes>
@@
 <attribute name="VALUE" x="70.649" y="1.795" size="1.27" layer="27" ratio="10" rot="R270"/>
 </element>
+<element name="BLAU" library="pinhead" library_urn="urn:adsk.eagle:library:325" package="1X01" package3d_urn="urn:adsk.eagle:package:22485/2" value="" x="11.1" y="6.1" smashed="yes">
+<attribute name="NAME" x="10.4462" y="5.2712" size="0.6096" layer="25" ratio="10" rot="R180"/>
+<attribute name="POPULARITY" value="64" x="11.1" y="6.1" size="1.778" layer="27" display="off"/>
+<attribute name="VALUE" x="9.83" y="2.925" size="1.27" layer="27"/>
+</element>
 </elements>
 <signals>
@@
 <wire x1="28.85335" y1="7.5048" x2="30.35815" y2="6" width="0.1524" layer="16"/>
 <wire x1="13.5634" y1="6.359" x2="13.5634" y2="7.45845625" width="0.1524" layer="16"/>
-<wire x1="1.0317625" y1="6.359" x2="13.5634" y2="6.359" width="0.1524" layer="16"/>
+<wire x1="1.0317625" y1="6.359" x2="11.359" y2="6.359" width="0.1524" layer="16"/>
+<wire x1="11.359" y1="6.359" x2="13.5634" y2="6.359" width="0.1524" layer="16"/>
 <wire x1="1.4" y1="2.93" x2="1.4" y2="4.2127625" width="0.1524" layer="16"/>
 <wire x1="1.4" y1="4.2127625" x2="0.511" y2="5.1017625" width="0.1524" layer="16"/>
@@
 <via x="42.7" y="5.9614" extent="1-16" drill="0.35"/>
 <wire x1="42.7" y1="5.9614" x2="42.7" y2="5.7" width="0.1524" layer="1"/>
+<contactref element="BLAU" pad="1"/>
+<wire x1="11.1" y1="6.1" x2="11.359" y2="6.359" width="0.1524" layer="16"/>
 </signal>
 <signal name="N$2">
@@
 <contactref element="TR-L-2" pad="1"/>
 <contactref element="D2" pad="A"/>
-<wire x1="5.87" y1="1.37" x2="7.64868125" y2="1.37" width="1.27" layer="1"/>
 <wire x1="14.8" y1="3.345" x2="7.845" y2="3.345" width="1.016" layer="1"/>
 <wire x1="7.845" y1="3.345" x2="5.87" y2="1.37" width="1.016" layer="1"/>
@@
 <contactref element="TR-R-2" pad="1"/>
 <contactref element="D3" pad="A"/>
-<wire x1="5.87" y1="6.65" x2="7.62868125" y2="6.65" width="1.27" layer="1"/>
 <wire x1="14.8" y1="4.615" x2="7.905" y2="4.615" width="1.016" layer="1"/>
 <wire x1="7.905" y1="4.615" x2="5.87" y2="6.65" width="1.016" layer="1"/>
