File: loc-decoder/Roco/BR215/br215.sch (EAGLE design)
At the start: 13 parts

Commit message: misc
Parts:
- added BLAU: (no value), pinhead:PINHD-1X1
Connections:
- net N$1: now also BLAU.1
Other:
- note added: "optional"
